File: MaxDC.kicad_pcb (KiCad board)
At the start: 2 copper layers, 99.5 x 100 mm, 34 parts, among them J1 L N E, J2 Screw_Terminal_01x04, T2 70063K

Commit message: Add files via upload
Parts:
- removed 240VAC: Symbol_HV_Type1_CopperTop_Small, Symbol:Symbol_Highvoltage_Type1_CopperTop_Small
- moved C6 3.90 mm to (162.5, 140.1)
- moved G*** 1.04 mm to (179.7, 89.0)
- moved C1 1.03 mm to (131.0, 142.0)
- moved C4 1.03 mm to (143.0, 142.0)
- moved C7 1.03 mm to (155.0, 142.0)
Routing:
- net T2: track 26.2 -> 22.5 mm, vias 2 -> 1
- net T1: track 19.8 -> 17.7 mm
Other:
- board text added: "E"
- board text added: "L"
- board text added: "MaxDC 0.3 Andrew Fischer 05022023 License: Creative Commons CC BY-NC 4.0 creativecommons.org/licenses/by-nc/4.0/"
- board text added: "N"
- board text removed: "MaxDC 0.3 Andrew Fischer 28012023 License: Creative Commons CC BY-NC 4.0 creativecommons.org/licenses/by-nc/4.0/"
